Commit message: Added robot model and early structure of the code

File: urdf/robot.xacro (robot description, xacro)
@@ -1,5 +1,5 @@
 <?xml version="1.0"?>
-<robot xmlns:xacro="http://www.ros.org/wiki/xacro" name="robot2_laser_xacro">
-<xacro:include filename="$(find planning)/urdf/robot2_laser.gazebo"/>
+<robot xmlns:xacro="http://www.ros.org/wiki/xacro" name="robot_xacro">
+<xacro:include filename="$(find exp_assignment3)/urdf/robot.gazebo"/>
 	<xacro:property name="length_wheel" value="0.02" />
 	<xacro:property name="radius_wheel" value="0.05" />
@@ -51,5 +51,5 @@
     <collision name="collision_chassis">
       <geometry>
-        <box size="0.25 0.15 0.035"/>
+        <box size="0.25 0.15 0.05"/>
       </geometry>
     </collision>
@@ -57,5 +57,5 @@
       <origin rpy="0 0 0" xyz="0 0 0"/>
       <geometry>
-        <box size="0.25 0.15 0.035"/>
+        <box size="0.25 0.15 0.05"/>
       </geometry>
       <material name="blue"/>
@@ -143,3 +143,30 @@
 	    <child link="hokuyo_link"/>
 	 </joint>
+  <!-- camera -->
+  <link name="camera_link">
+	    <collision>
+	      <origin xyz="-0.025 0 0.05" rpy="0 0 0"/>
+	      <geometry>
+		      <box size="0.05 0.05 0.05"/>
+	      </geometry>
+	    </collision>
+	    <visual>
+	      <origin xyz="-0.025 0 0.05" rpy="0 0 0"/>
+	      <geometry>
+		      <box size="0.05 0.05 0.05"/>
+	      </geometry>
+	      <material name="grey"/>
+	    </visual>
+	    <inertial>
+	      <mass value="1e-5" />
+	      <origin xyz="0 0 0" rpy="0 0 0"/>
+	      <inertia ixx="1e-6" ixy="0" ixz="0" iyy="1e-6" iyz="0" izz="1e-6" />
+	    </inertial>
+  </link>
+  <joint name="camera_joint" type="fixed">
+	    <axis xyz="0 1 0" />
+	    <origin xyz="0.15 0 0.0" rpy="0 0 0"/>
+      <child link="camera_link"/>
+	    <parent link="link_chassis"/>
+	</joint>
 </robot>

Commit message: Initial implementation of Normal and Sleep behaviour

File: urdf/robot.xacro (robot description, xacro)
@@ -100,4 +100,5 @@
     </visual>
   </link>
+<!--
   <link name="link_right_wheel_2">
     <xacro:default_inertial mass="0.2"/>
@@ -124,6 +125,7 @@
     </visual>
   </link>
+-->
   <joint name="joint_right_wheel" type="continuous">
-    <origin rpy="0 0 0" xyz="-0.025 0.075 0"/>
+    <origin rpy="0 0 0" xyz="-0.075 0.075 0"/>
     <child link="link_right_wheel"/>
     <parent link="link_chassis"/>
@@ -133,5 +135,5 @@
   </joint>
   <joint name="joint_left_wheel" type="continuous">
-    <origin rpy="0 0 0" xyz="-0.025 -0.075 0"/>
+    <origin rpy="0 0 0" xyz="-0.075 -0.075 0"/>
     <child link="link_left_wheel"/>
     <parent link="link_chassis"/>
@@ -140,5 +142,5 @@
     <joint_properties damping="1.0" friction="1.0"/>
   </joint>
-  <joint name="joint_right_wheel_2" type="continuous">
+  <!--<joint name="joint_right_wheel_2" type="continuous">
     <origin rpy="0 0 0" xyz="-0.075 0.075 0"/>
     <child link="link_right_wheel_2"/>
@@ -156,4 +158,5 @@
     <joint_properties damping="1.0" friction="1.0"/>
   </joint>
+-->
   <!-- laser -->
   <link name="hokuyo_link">
@@ -198,5 +201,5 @@
 		      <box size="0.05 0.05 0.05"/>
 	      </geometry>
-	      <material name="grey"/>
+	      <material name="red"/>
 	    </visual>
 	    <inertial>

Commit message: Added Track Substate

File: urdf/robot.xacro (robot description, xacro)
@@ -127,5 +127,5 @@
 -->
   <joint name="joint_right_wheel" type="continuous">
-    <origin rpy="0 0 0" xyz="-0.075 0.075 0"/>
+    <origin rpy="0 0 0" xyz="-0.025 0.075 0"/>
     <child link="link_right_wheel"/>
     <parent link="link_chassis"/>
@@ -135,5 +135,5 @@
   </joint>
   <joint name="joint_left_wheel" type="continuous">
-    <origin rpy="0 0 0" xyz="-0.075 -0.075 0"/>
+    <origin rpy="0 0 0" xyz="-0.025 -0.075 0"/>
     <child link="link_left_wheel"/>
     <parent link="link_chassis"/>
